File: hw4/hw4.2/hw4.2.kicad_sch (KiCad schematic)
At the start: 23 parts, among them J1 BATTERY, J2 CP2102, J3 Conn_01x12_Pin, J4 Conn_01x12_Pin, SW1 SW_Push, SW2 SW_Push, SW4 SW_silde, U2 AP7384-33V

Commit message: Starting work on HW2.
Parts:
- C1, C2, C3, C5: footprint (none) -> Capacitor_THT:C_Disc_D5.1mm_W3.2mm_P5.00mm
- C4, C6: footprint (none) -> Capacitor_THT:C_Disc_D3.4mm_W2.1mm_P2.50mm
- D1, D2, D3: footprint (none) -> LED_THT:LED_D3.0mm
- J1: footprint (none) -> Connector_PinSocket_2.54mm:PinSocket_1x02_P2.54mm_Vertical
- J2: footprint (none) -> Connector_PinSocket_2.54mm:PinSocket_1x06_P2.54mm_Vertical
- J3: value Conn_01x12_Pin -> LEFT; footprint (none) -> Connector_PinSocket_2.54mm:PinSocket_1x12_P2.54mm_Vertical
- J4: value Conn_01x12_Pin -> RIGHT; footprint (none) -> Connector_PinSocket_2.54mm:PinSocket_1x12_P2.54mm_Vertical
- R1, R2, R3, R4, R5: footprint (none) -> Resistor_THT:R_Axial_DIN0207_L6.3mm_D2.5mm_P7.62mm_Horizontal
- SW1: value SW_Push -> MCLR; footprint (none) -> pic32:pb
- SW2: value SW_Push -> USER; footprint (none) -> pic32:pb
- SW4: footprint (none) -> pic32:slidesw2
- U1: footprint (none) -> Package_DIP:DIP-28_W7.62mm_Socket
- U2: value AP7384-33V -> AP7381-33V; footprint (none) -> Package_TO_SOT_THT:TO-92L_Inline
Connections:
- net YeELLOW is gone; now on net YELLOW: J3.8 (Pin_8)
- net +3.3V: now also C1.1, C2.1, D1.2 (A), U2.1 (VO)
- net GND1: now reaches C4.2, U1.27 (AVSS)
- net GND1: now also C1.2, C2.2, C3.2, C5.2, C6.2, J1.2 (Pin_2), J2.6 (Pin_6), J3.12 (Pin_12), J4.12 (Pin_12), R1.2, SW1.1, SW2.1, U1.19 (VSS), U1.8 (VSS), U2.2 (GND)
